File: cad/Stirplate.brd (EAGLE design)
At the start: 42.5 x 43.2 mm, 14 parts, among them IC1 DS18B20, IC3 7505

Commit message: Refactor
Parts:
- renumbered IC1 to U2, IC3 to U3, U$1 to U1
Changed lines of the file:
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@@
 </autorouter>
 <elements>
-<element name="U$1" library="diy-modules" package="WEMOS-D1-MINI" value="WEMOS-D1-MINI" x="21.59" y="20.955" smashed="yes">
+<element name="U1" library="diy-modules" package="WEMOS-D1-MINI" value="WEMOS-D1-MINI" x="21.59" y="20.955" smashed="yes">
 <attribute name="NAME" x="20.955" y="32.7025" size="1.27" layer="25"/>
 <attribute name="VALUE" x="35.56" y="34.29" size="1.27" layer="27"/>
@@
 </element>
 <element name="U$3" library="holes" package="3,0" value="" x="22.5425" y="38.735" smashed="yes"/>
-<element name="IC1" library="1wire" package="TO92-" value="DS18B20" x="38.1" y="35.56" smashed="yes" rot="R270">
+<element name="U2" library="1wire" package="TO92-" value="DS18B20" x="38.1" y="35.56" smashed="yes" rot="R270">
 <attribute name="NAME" x="36.0045" y="34.29" size="1.27" layer="25" ratio="10" rot="R90"/>
 <attribute name="VALUE" x="34.798" y="38.1" size="1.27" layer="27" ratio="10" rot="R270"/>
 </element>
-<element name="IC3" library="v-reg" package="78XXL" value="7505" x="34.29" y="5.08" smashed="yes" rot="R90">
+<element name="U3" library="v-reg" package="78XXL" value="7505" x="34.29" y="5.08" smashed="yes" rot="R90">
 <attribute name="NAME" x="19.05" y="3.175" size="1.778" layer="25" ratio="10" rot="R90"/>
 <attribute name="VALUE" x="31.75" y="1.143" size="1.778" layer="27" ratio="10" rot="R90"/>
@@
 <signals>
 <signal name="3V3">
-<contactref element="U$1" pad="JP1.8"/>
+<contactref element="U1" pad="JP1.8"/>
 </signal>
 <signal name="N$1">
-<contactref element="U$1" pad="JP1.2"/>
+<contactref element="U1" pad="JP1.2"/>
 <contactref element="R3" pad="2"/>
 <wire x1="10.16" y1="27.94" x2="21.59" y2="27.94" width="0.6096" layer="1"/>
@@
 </signal>
 <signal name="+5V">
-<contactref element="U$1" pad="JP2.8"/>
+<contactref element="U1" pad="JP2.8"/>
 <contactref element="R1" pad="2"/>
 <contactref element="R2" pad="2"/>
@@
 <wire x1="12.7" y1="31.115" x2="12.7" y2="32.385" width="0.6096" layer="16"/>
 <wire x1="12.7" y1="32.385" x2="12.065" y2="33.02" width="0.6096" layer="16"/>
-<contactref element="IC1" pad="3"/>
+<contactref element="U2" pad="3"/>
 <wire x1="17.78" y1="17.78" x2="19.685" y2="17.78" width="0.6096" layer="16"/>
 <wire x1="19.685" y1="17.78" x2="20.32" y2="17.78" width="0.6096" layer="16"/>
 <wire x1="20.32" y1="17.78" x2="20.32" y2="18.415" width="0.6096" layer="16"/>
-<contactref element="IC3" pad="OUT"/>
+<contactref element="U3" pad="OUT"/>
 <wire x1="20.32" y1="18.415" x2="20.32" y2="22.86" width="0.6096" layer="16"/>
 <wire x1="20.32" y1="23.495" x2="20.32" y2="22.86" width="0.6096" layer="16"/>
@@
 <signal name="GND">
 <contactref element="R3" pad="1"/>
-<contactref element="U$1" pad="JP2.7"/>
+<contactref element="U1" pad="JP2.7"/>
 <contactref element="SV1" pad="1"/>
 <contactref element="C3" pad="-"/>
@@
 <vertex x="0" y="43.18"/>
 </polygon>
-<contactref element="IC1" pad="1"/>
-<contactref element="IC3" pad="GND"/>
+<contactref element="U2" pad="1"/>
+<contactref element="U3" pad="GND"/>
 </signal>
 <signal name="+12V">
@@
 <contactref element="X1" pad="1"/>
 <contactref element="SV1" pad="2"/>
-<contactref element="IC3" pad="IN"/>
+<contactref element="U3" pad="IN"/>
 <wire x1="38.1" y1="2.54" x2="29.845" y2="2.54" width="0.6096" layer="16"/>
 <wire x1="12.065" y1="2.54" x2="5.08" y2="2.54" width="0.6096" layer="16"/>
@@
 </signal>
 <signal name="N$5">
-<contactref element="U$1" pad="JP1.4"/>
+<contactref element="U1" pad="JP1.4"/>
 <contactref element="SV1" pad="4"/>
 <wire x1="5.08" y1="22.86" x2="10.16" y2="22.86" width="0.6096" layer="16"/>
 </signal>
 <signal name="N$4">
-<contactref element="U$1" pad="JP1.5"/>
+<contactref element="U1" pad="JP1.5"/>
 <contactref element="SV1" pad="3"/>
 <contactref element="R2" pad="1"/>
@@
 </signal>
 <signal name="N$8">
-<contactref element="U$1" pad="JP2.4"/>
+<contactref element="U1" pad="JP2.4"/>
 <contactref element="SV2" pad="3"/>
 <wire x1="33.02" y1="22.86" x2="26.035" y2="22.86" width="0.6096" layer="16"/>
@@
 </signal>
 <signal name="N$9">
-<contactref element="U$1" pad="JP2.3"/>
+<contactref element="U1" pad="JP2.3"/>
 <contactref element="SV2" pad="4"/>
 <wire x1="5.08" y1="38.1" x2="15.875" y2="38.1" width="0.6096" layer="16"/>
@@
 </signal>
 <signal name="1W">
-<contactref element="U$1" pad="JP2.6"/>
-<contactref element="IC1" pad="2"/>
+<contactref element="U1" pad="JP2.6"/>
+<contactref element="U2" pad="2"/>
 <wire x1="33.02" y1="17.78" x2="35.56" y2="17.78" width="0.6096" layer="16"/>
 <wire x1="35.56" y1="17.78" x2="36.195" y2="18.415" width="0.6096" layer="16"/>
