File: cad/Stirplate.brd (EAGLE design)
At the start: 43.8 x 43.2 mm, 13 parts, among them U1 WEMOS-D1-MINI, U2 DS18B20, U4 PMX42_LD1086VXX-H

Commit message: Testing v1.5.1
Routing:
- net +5V: track 106.4 -> 98.7 mm
Changed lines of the file:
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@@
 <layer number="46" name="Milling" color="3" fill="1" visible="yes" active="yes"/>
 <layer number="47" name="Measures" color="7" fill="1" visible="yes" active="yes"/>
-<layer number="48" name="Document" color="7" fill="1" visible="yes" active="yes"/>
+<layer number="48" name="Document" color="7" fill="1" visible="no" active="yes"/>
 <layer number="49" name="Reference" color="7" fill="1" visible="yes" active="yes"/>
 <layer number="50" name="dxf" color="7" fill="1" visible="no" active="no"/>
@@
 </signal>
 <signal name="N$1">
-<contactref element="U1" pad="JP1.2"/>
 <contactref element="R3" pad="2"/>
 <wire x1="10.16" y1="27.94" x2="21.59" y2="27.94" width="0.6096" layer="1"/>
@@
 <wire x1="36.195" y1="22.225" x2="36.195" y2="31.75" width="0.6096" layer="1"/>
 <wire x1="36.195" y1="31.75" x2="35.56" y2="32.385" width="0.6096" layer="1"/>
+<contactref element="U1" pad="JP1.2"/>
 </signal>
 <signal name="N$2">
@@
 </signal>
 <signal name="+5V">
-<contactref element="U1" pad="JP2.8"/>
 <contactref element="R1" pad="2"/>
 <contactref element="R2" pad="2"/>
@@
 <wire x1="12.7" y1="32.385" x2="12.065" y2="33.02" width="0.6096" layer="16"/>
 <contactref element="U2" pad="3"/>
-<wire x1="19.685" y1="17.78" x2="20.32" y2="17.78" width="0.6096" layer="16"/>
 <wire x1="20.32" y1="17.78" x2="20.32" y2="18.415" width="0.6096" layer="16"/>
 <wire x1="20.32" y1="18.415" x2="20.32" y2="22.86" width="0.6096" layer="16"/>
@@
 <wire x1="20.32" y1="29.845" x2="19.685" y2="30.48" width="0.6096" layer="16"/>
 <wire x1="19.685" y1="30.48" x2="16.51" y2="30.48" width="0.6096" layer="16"/>
-<wire x1="20.32" y1="17.145" x2="19.685" y2="17.78" width="0.6096" layer="16"/>
-<wire x1="19.685" y1="17.78" x2="20.32" y2="18.415" width="0.6096" layer="16"/>
-<wire x1="38.1" y1="12.065" x2="38.1" y2="12.7" width="0.6096" layer="16"/>
-<wire x1="38.1" y1="12.7" x2="38.1" y2="13.335" width="0.6096" layer="16"/>
 <wire x1="38.1" y1="13.335" x2="38.1" y2="33.02" width="0.6096" layer="16"/>
 <wire x1="27.305" y1="20.32" x2="27.305" y2="12.7" width="0.6096" layer="16"/>
-<wire x1="27.94" y1="13.335" x2="27.94" y2="12.7" width="0.6096" layer="16"/>
-<wire x1="27.305" y1="12.7" x2="27.94" y2="13.335" width="0.6096" layer="16"/>
-<wire x1="27.94" y1="13.335" x2="28.575" y2="12.7" width="0.6096" layer="16"/>
 <contactref element="R4" pad="2"/>
 <wire x1="27.305" y1="20.32" x2="30.48" y2="20.32" width="0.6096" layer="16"/>
 <wire x1="33.02" y1="12.7" x2="37.465" y2="12.7" width="0.6096" layer="16"/>
-<wire x1="37.465" y1="12.7" x2="38.1" y2="12.7" width="0.6096" layer="16"/>
-<wire x1="38.1" y1="12.065" x2="37.465" y2="12.7" width="0.6096" layer="16"/>
 <wire x1="37.465" y1="12.7" x2="38.1" y2="13.335" width="0.6096" layer="16"/>
 <contactref element="U4" pad="2"/>
@@
 <wire x1="40.62" y1="5.715" x2="38.481" y2="5.715" width="0.508" layer="16"/>
 <wire x1="34.925" y1="10.795" x2="40.62" y2="10.795" width="0.508" layer="16"/>
+<contactref element="U1" pad="JP2.8"/>
 </signal>
 <signal name="GND">
@@
 </signal>
 <signal name="N$5">
-<contactref element="U1" pad="JP1.4"/>
 <contactref element="SV1" pad="4"/>
 <wire x1="5.08" y1="22.86" x2="10.16" y2="22.86" width="0.6096" layer="16"/>
+<contactref element="U1" pad="JP1.4"/>
 </signal>
 <signal name="N$4">
-<contactref element="U1" pad="JP1.5"/>
 <contactref element="SV1" pad="3"/>
 <contactref element="R2" pad="1"/>
 <wire x1="16.51" y1="20.32" x2="10.16" y2="20.32" width="0.6096" layer="16"/>
 <wire x1="10.16" y1="20.32" x2="5.08" y2="20.32" width="0.6096" layer="16"/>
+<contactref element="U1" pad="JP1.5"/>
 </signal>
 <signal name="N$8">
-<contactref element="U1" pad="JP2.4"/>
 <contactref element="SV2" pad="3"/>
 <wire x1="33.02" y1="22.86" x2="26.035" y2="22.86" width="0.6096" layer="16"/>
@@
 <wire x1="15.24" y1="32.385" x2="22.86" y2="32.385" width="0.6096" layer="16"/>
 <wire x1="22.86" y1="32.385" x2="23.495" y2="31.75" width="0.6096" layer="16"/>
+<contactref element="U1" pad="JP2.4"/>
 </signal>
 <signal name="N$9">
-<contactref element="U1" pad="JP2.3"/>
 <contactref element="SV2" pad="4"/>
 <wire x1="5.08" y1="38.1" x2="15.875" y2="38.1" width="0.6096" layer="16"/>
@@
 <wire x1="17.145" y1="33.655" x2="24.765" y2="33.655" width="0.6096" layer="16"/>
 <wire x1="24.765" y1="33.655" x2="25.4" y2="33.02" width="0.6096" layer="16"/>
+<contactref element="U1" pad="JP2.3"/>
 </signal>
 <signal name="1W">
-<contactref element="U1" pad="JP2.6"/>
 <contactref element="U2" pad="2"/>
 <wire x1="33.02" y1="17.78" x2="35.56" y2="17.78" width="0.6096" layer="16"/>
@@
 <wire x1="35.56" y1="33.655" x2="36.195" y2="34.29" width="0.6096" layer="16"/>
 <wire x1="36.195" y1="33.02" x2="35.56" y2="33.655" width="0.6096" layer="16"/>
+<contactref element="U1" pad="JP2.6"/>
 </signal>
 </signals>

Commit message: Updated readme
Routing:
- net N$2: track 35.2 -> 32.9 mm
