File: cad/Stirplate.sch (EAGLE design)
At the start: 13 parts, among them IC1 DS18B20, IC3 7505

Commit message: Refactor
Parts:
- renumbered IC1 to U2, IC3 to U3, U$1 to U1
Other:
- note added: "GPIO5 = SCL = D1 GPIO4 = SDA = D2 GPIO2 = TEMP = D4 GPIO12 = Tacto = D6 GPIO14 = PWM = D5"
- note removed: "GPIO5 = SCL = D1 GPIO4= SDA = D2 GPIO12= Tacto = D6 GPIO14 = PWM = D5"
Changed lines of the file:
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@@
 </classes>
 <parts>
-<part name="U$1" library="diy-modules" deviceset="WEMOS-D1-MINI" device=""/>
+<part name="U1" library="diy-modules" deviceset="WEMOS-D1-MINI" device=""/>
 <part name="C1" library="rcl" deviceset="C-EU" device="050-025X075" value="100n"/>
 <part name="C2" library="rcl" deviceset="CPOL-EU" device="E2.5-5" value="10u"/>
@@
 <part name="P+5" library="supply1" deviceset="+5V" device=""/>
 <part name="SUPPLY10" library="supply2" deviceset="GND" device="" value=""/>
-<part name="IC1" library="1wire" deviceset="DS18B20" device=""/>
-<part name="IC3" library="v-reg" deviceset="78XXL" device="" value="7505"/>
+<part name="U2" library="1wire" deviceset="DS18B20" device=""/>
+<part name="U3" library="v-reg" deviceset="78XXL" device="" value="7505"/>
 <part name="R4" library="rcl" deviceset="R-EU_" device="0207/10" value="4.7K"/>
 <part name="P+9" library="supply1" deviceset="+5V" device=""/>
@@
 <sheet>
 <plain>
-<text x="60.96" y="10.16" size="1.778" layer="91">GPIO5 = SCL = D1
-GPIO4= SDA = D2
-GPIO12= Tacto = D6
+<text x="58.42" y="5.08" size="1.778" layer="91">GPIO5   = SCL = D1
+GPIO4   = SDA = D2
+GPIO2   = TEMP = D4
+GPIO12 = Tacto = D6
 GPIO14 = PWM = D5</text>
 </plain>
 <instances>
-<instance part="U$1" gate="G$1" x="71.12" y="40.64" smashed="yes">
+<instance part="U1" gate="G$1" x="71.12" y="40.64" smashed="yes">
 <attribute name="NAME" x="58.42" y="66.04" size="1.778" layer="95"/>
 <attribute name="VALUE" x="58.42" y="63.5" size="1.778" layer="96"/>
@@
 <attribute name="VALUE" x="117.475" y="37.465" size="1.778" layer="96"/>
 </instance>
-<instance part="IC1" gate="G$1" x="104.14" y="35.56" smashed="yes" rot="MR0">
+<instance part="U2" gate="G$1" x="104.14" y="35.56" smashed="yes" rot="MR0">
 <attribute name="NAME" x="114.3" y="35.56" size="1.27" layer="95" rot="MR0" align="bottom-right"/>
 <attribute name="VALUE" x="114.3" y="33.02" size="1.27" layer="96" rot="MR0" align="bottom-right"/>
 </instance>
-<instance part="IC1" gate="P" x="109.22" y="35.56" smashed="yes">
+<instance part="U2" gate="P" x="109.22" y="35.56" smashed="yes">
 <attribute name="NAME" x="111.125" y="40.005" size="1.778" layer="95" font="vector"/>
 </instance>
-<instance part="IC3" gate="A" x="38.1" y="91.44" smashed="yes">
+<instance part="U3" gate="A" x="38.1" y="91.44" smashed="yes">
 <attribute name="NAME" x="40.64" y="83.82" size="1.778" layer="95"/>
 <attribute name="VALUE" x="40.64" y="81.28" size="1.778" layer="96"/>
@@
 <net name="N$1" class="0">
 <segment>
-<pinref part="U$1" gate="G$1" pin="A0"/>
+<pinref part="U1" gate="G$1" pin="A0"/>
 <pinref part="R3" gate="G$1" pin="S"/>
 <wire x1="53.34" y1="48.26" x2="45.72" y2="48.26" width="0.1524" layer="91"/>
@@
 <net name="+5V" class="0">
 <segment>
-<pinref part="U$1" gate="G$1" pin="5V"/>
+<pinref part="U1" gate="G$1" pin="5V"/>
 <wire x1="88.9" y1="33.02" x2="93.98" y2="33.02" width="0.1524" layer="91"/>
 <wire x1="93.98" y1="33.02" x2="93.98" y2="71.12" width="0.1524" layer="91"/>
@@
 <pinref part="P+3" gate="1" pin="+5V"/>
 <wire x1="109.22" y1="43.18" x2="109.22" y2="71.12" width="0.1524" layer="91"/>
-<pinref part="IC1" gate="P" pin="VDD"/>
+<pinref part="U2" gate="P" pin="VDD"/>
 </segment>
 <segment>
@@
 <junction x="48.26" y="91.44"/>
 <pinref part="P+6" gate="1" pin="+5V"/>
-<pinref part="IC3" gate="A" pin="OUT"/>
+<pinref part="U3" gate="A" pin="OUT"/>
 </segment>
 <segment>
@@
 </segment>
 <segment>
-<pinref part="U$1" gate="G$1" pin="GND"/>
+<pinref part="U1" gate="G$1" pin="GND"/>
 <wire x1="88.9" y1="35.56" x2="96.52" y2="35.56" width="0.1524" layer="91"/>
 <wire x1="96.52" y1="35.56" x2="96.52" y2="27.94" width="0.1524" layer="91"/>
@@
 <wire x1="38.1" y1="83.82" x2="38.1" y2="81.28" width="0.1524" layer="91"/>
 <pinref part="SUPPLY7" gate="GND" pin="GND"/>
-<pinref part="IC3" gate="A" pin="GND"/>
+<pinref part="U3" gate="A" pin="GND"/>
 </segment>
 <segment>
@@
 <segment>
 <pinref part="SUPPLY3" gate="GND" pin="GND"/>
-<pinref part="IC1" gate="P" pin="GND"/>
+<pinref part="U2" gate="P" pin="GND"/>
 </segment>
 </net>
@@
 <pinref part="P+7" gate="1" pin="+12V"/>
 <pinref part="X1" gate="-1" pin="KL"/>
-<pinref part="IC3" gate="A" pin="IN"/>
+<pinref part="U3" gate="A" pin="IN"/>
 </segment>
 <segment>
@@
 <segment>
 <wire x1="45.72" y1="38.1" x2="45.72" y2="43.18" width="0.1524" layer="91"/>
-<pinref part="U$1" gate="G$1" pin="D5"/>
+<pinref part="U1" gate="G$1" pin="D5"/>
 <wire x1="45.72" y1="43.18" x2="53.34" y2="43.18" width="0.1524" layer="91"/>
 <pinref part="SV1" gate="1" pin="4"/>
@@
 <net name="N$4" class="0">
 <segment>
-<pinref part="U$1" gate="G$1" pin="D6"/>
+<pinref part="U1" gate="G$1" pin="D6"/>
 <wire x1="53.34" y1="40.64" x2="25.4" y2="40.64" width="0.1524" layer="91"/>
 <pinref part="SV1" gate="1" pin="3"/>
@@
 <net name="N$8" class="0">
 <segment>
-<pinref part="U$1" gate="G$1" pin="D2"/>
+<pinref part="U1" gate="G$1" pin="D2"/>
 <wire x1="88.9" y1="43.18" x2="104.14" y2="43.18" width="0.1524" layer="91"/>
 <wire x1="104.14" y1="43.18" x2="104.14" y2="48.26" width="0.1524" layer="91"/>
@@
 <net name="N$9" class="0">
 <segment>
-<pinref part="U$1" gate="G$1" pin="D1"/>
+<pinref part="U1" gate="G$1" pin="D1"/>
 <pinref part="SV2" gate="1" pin="4"/>
 <wire x1="88.9" y1="45.72" x2="121.92" y2="45.72" width="0.1524" layer="91"/>
@@
 <segment>
 <wire x1="101.6" y1="35.56" x2="101.6" y2="38.1" width="0.1524" layer="91"/>
-<pinref part="U$1" gate="G$1" pin="D4"/>
+<pinref part="U1" gate="G$1" pin="D4"/>
 <wire x1="88.9" y1="38.1" x2="101.6" y2="38.1" width="0.1524" layer="91"/>
-<pinref part="IC1" gate="G$1" pin="1W"/>
+<pinref part="U2" gate="G$1" pin="1W"/>
 <wire x1="101.6" y1="35.56" x2="104.14" y2="35.56" width="0.1524" layer="91"/>
 <pinref part="R4" gate="G$1" pin="1"/>
